File: harware/fleemo.sch (KiCad schematic (older format))
At the start: 48 parts, among them P1 CONN_01X02, P2 CONN_01X03, P3 RESET_PAD, Q1 STD2HNK60Z-1, U1 AMS1117, U2 wurth-750312723, U3 UCC28700, U4 STM32F030F4Px, U5 FLEEMO, Y1 8Mhz

Commit message: add some more footprint
Parts:
- R3: footprint (none) -> Resistors_ThroughHole:Resistor_Horizontal_RM15mm
- U2: footprint (none) -> lib:750312723
- U4: footprint TSSOP20 -> lib:TSSOP20
Changed lines of the file:
@@
 F 0 "U2" H 8050 2800 60  0000 C CNN
 F 1 "wurth-750312723" H 8650 2400 60  0000 C CNN
-F 2 "" H 8150 1900 60  0001 C CNN
+F 2 "lib:750312723" H 8150 1900 60  0001 C CNN
 F 3 "" H 8150 1900 60  0000 C CNN
 	1    8150 1900
@@
 F 0 "R3" V 2950 2550 50  0000 L CNN
 F 1 "10" V 3150 2550 50  0000 L CNN
-F 2 "" H 3050 2600 50  0001 C CNN
+F 2 "Resistors_ThroughHole:Resistor_Horizontal_RM15mm" H 3050 2600 50  0001 C CNN
 F 3 "" H 3050 2600 50  0000 C CNN
 	1    3050 2600
@@
 F 0 "U4" H 6900 6025 50  0000 L BNN
 F 1 "STM32F030F4Px" H 10100 6025 50  0000 R BNN
-F 2 "TSSOP20" H 10100 5975 50  0000 R TNN
+F 2 "lib:TSSOP20" H 10100 5975 50  0000 R TNN
 F 3 "" H 8500 5100 50  0000 C CNN
 	1    8500 5100

Commit message: adding more footprint
Parts:
- P1: value CONN_01X02 -> AC_IN; footprint (none) -> lib:AC_IN
- P2: value CONN_01X03 -> PROGRAM; footprint (none) -> Pin_Headers:Pin_Header_Straight_1x03
- P3: footprint (none) -> Pin_Headers:Pin_Header_Straight_1x01
- U5: footprint (none) -> lib:fleemo
Changed lines of the file:
@@
 P 2650 2650
 F 0 "P1" H 2650 2800 50  0000 C CNN
-F 1 "CONN_01X02" V 2750 2650 50  0000 C CNN
-F 2 "" H 2650 2650 50  0001 C CNN
+F 1 "AC_IN" V 2750 2650 50  0000 C CNN
+F 2 "lib:AC_IN" H 2650 2650 50  0001 C CNN
 F 3 "" H 2650 2650 50  0000 C CNN
 	1    2650 2650
@@
 P 5550 4100
 F 0 "P2" H 5550 4300 50  0000 C CNN
-F 1 "CONN_01X03" H 5450 3900 50  0000 C CNN
-F 2 "" H 5550 4100 50  0001 C CNN
+F 1 "PROGRAM" H 5450 3900 50  0000 C CNN
+F 2 "Pin_Headers:Pin_Header_Straight_1x03" H 5550 4100 50  0001 C CNN
 F 3 "" H 5550 4100 50  0000 C CNN
 	1    5550 4100
@@
 F 0 "P3" H 6400 4600 50  0000 C CNN
 F 1 "RESET_PAD" H 6500 4400 50  0000 C CNN
-F 2 "" H 6400 4500 50  0001 C CNN
+F 2 "Pin_Headers:Pin_Header_Straight_1x01" H 6400 4500 50  0001 C CNN
 F 3 "" H 6400 4500 50  0000 C CNN
 	1    6400 4500
@@
 F 0 "U5" H 5350 5900 60  0000 C CNN
 F 1 "FLEEMO" H 5450 5350 60  0000 C CNN
-F 2 "" H 5450 5350 60  0001 C CNN
+F 2 "lib:fleemo" H 5450 5350 60  0001 C CNN
 F 3 "" H 5450 5350 60  0000 C CNN
 	1    5450 5350
